File: usb_to_ttl-ch340/usb_to_ttl-ch340.sch (KiCad schematic (older format))
At the start: 20 parts, among them J1 USB_OTG, J2 6_pin_header, U1 CH340G, Y1 12MHz

Commit message: güncelleme
Parts:
- removed D1, D2: LL4148, Diode_SMD:D_MiniMELF, symbol Diode:LL4148
Connections:
- net reset: now also J2.5
Changed lines of the file:
@@
-$EndComp
-$Comp
-L Diode:LL4148 D1
-U 1 1 6132AA51
-P 8600 2700
-F 0 "D1" H 8600 2483 50  0000 C CNN
-F 1 "LL4148" H 8600 2574 50  0000 C CNN
-F 2 "Diode_SMD:D_MiniMELF" H 8600 2525 50  0001 C CNN
-F 3 "http://www.vishay.com/docs/85557/ll4148.pdf" H 8600 2700 50  0001 C CNN
-	1    8600 2700
-	-1   0    0    1
-$EndComp
-$Comp
-L Diode:LL4148 D2
-U 1 1 6132B2F6
-P 9300 2700
-F 0 "D2" H 9300 2483 50  0000 C CNN
-F 1 "LL4148" H 9300 2574 50  0000 C CNN
-F 2 "Diode_SMD:D_MiniMELF" H 9300 2525 50  0001 C CNN
-F 3 "http://www.vishay.com/docs/85557/ll4148.pdf" H 9300 2700 50  0001 C CNN
-	1    9300 2700
-	-1   0    0    1
 $EndComp
 $Comp
@@
 Connection ~ 7450 2450
 Wire Wire Line
-	8050 2900 8050 2700
-Wire Wire Line
 	8050 3200 8050 3450
-Wire Wire Line
-	8450 2700 8050 2700
-Connection ~ 8050 2700
-Wire Wire Line
-	8050 2700 8050 2450
-Wire Wire Line
-	8750 2700 9150 2700
-Wire Wire Line
-	9450 2700 9850 2700
 Wire Wire Line
 	9850 2700 9850 3350
@@
 Wire Wire Line
 	9550 3400 10200 3400
+Wire Wire Line
+	8050 2450 8050 2900
+Text GLabel 9650 2700 0    50   Input ~ 0
+reset
+Wire Wire Line
+	9650 2700 9850 2700
 $EndSCHEMATC

Commit message: düzeltme3
Connections:
- net +5V: now also C1.1, D3.2 (A), J2.6, R1.1, R2.1, U1.16 (VCC)
Changed lines of the file:
@@
 Wire Wire Line
 	9650 2700 9850 2700
+$Comp
+L power:+5V #PWR?
+U 1 1 61377922
+P 7450 2300
+F 0 "#PWR?" H 7450 2150 50  0001 C CNN
+F 1 "+5V" H 7465 2473 50  0000 C CNN
+F 2 "" H 7450 2300 50  0001 C CNN
+F 3 "" H 7450 2300 50  0001 C CNN
+	1    7450 2300
+	1    0    0    -1
+$EndComp
+Wire Wire Line
+	7450 2300 7450 2450
 $EndSCHEMATC

Commit message: diffferential pair
Connections:
- net D+: now reaches J1.3 (D+), U1.5 (UD+)
- net D-: now reaches J1.2 (D-), U1.6 (UD-)
Changed lines of the file:
@@
 	9650 2700 9850 2700
 $Comp
-L power:+5V #PWR?
+L power:+5V #PWR0101
 U 1 1 61377922
 P 7450 2300
-F 0 "#PWR?" H 7450 2150 50  0001 C CNN
+F 0 "#PWR0101" H 7450 2150 50  0001 C CNN
 F 1 "+5V" H 7465 2473 50  0000 C CNN
 F 2 "" H 7450 2300 50  0001 C CNN
@@
 Wire Wire Line
 	7450 2300 7450 2450
+Text Label 2150 3300 0    50   ~ 0
+D+
+Text Label 2150 3400 0    50   ~ 0
+D-
 $EndSCHEMATC
