File: buck_converter/buck_converter.sch (KiCad schematic (older format))
At the start: 22 parts, among them Q1 IRF6641, U1 LM741, U2 LM741, U3 LM741, U4 LM741

Commit message: güncelleme
kontrol edilmeyecek de olsa hatalı olduğumu belirttiğiniz noktaları düzeltmeye çalıştım
Parts:
- removed R2, R3, R4, R5, R6, R7, R8: R, Resistor_SMD:R_0201_0603Metric, symbol Device:R
- removed U1, U2, U3, U4: LM741, opamp:lm741, symbol Amplifier_Operational:LM741
- removed v1: vin, klemens:2xKlemens, symbol 2xKlemens:klemens
- removed v2: load, klemens:2xKlemens, symbol 2xKlemens:klemens
- removed v3: signal, klemens:2xKlemens, symbol 2xKlemens:klemens
- removed v4: battery, klemens:2xKlemens, symbol 2xKlemens:klemens
- added BT1: 4V5, Battery:BatteryHolder_Keystone_2479_3xAAA, symbol Device:Battery
- added D2, D3: D, Diode_SMD:D_0201_0603Metric_Pad0.64x0.40mm_HandSolder, symbol Device:D
- added J1: Conn_01x02_Male, Connector_PinHeader_1.27mm:PinHeader_1x02_P1.27mm_Vertical, symbol Connector:Conn_01x02_Male
- added J2: Conn_01x02_Female, Connector_PinSocket_1.00mm:PinSocket_1x02_P1.00mm_Vertical, symbol Connector:Conn_01x02_Female
- added RV1: 100k, Potentiometer_SMD:Potentiometer_ACP_CA9-VSMD_Vertical_Hole, symbol Device:R_POT
- added U1: NE555D, Package_SO:SOIC-8_3.9x4.9mm_P1.27mm, symbol Timer:NE555D
- C1: value C -> 380uF
- C2: value C -> 10nF; footprint Capacitor_SMD:C_0504_1310Metric -> Capacitor_SMD:C_0504_1310Metric_Pad0.83x1.28mm_HandSolder
- C3: value C -> 1uF; footprint Capacitor_SMD:C_0504_1310Metric -> Capacitor_SMD:C_0504_1310Metric_Pad0.83x1.28mm_HandSolder
- L1: value INDUCTOR -> 100uH
- R1: value R -> 1k; footprint Resistor_SMD:R_0201_0603Metric -> Resistor_SMD:R_0402_1005Metric_Pad0.72x0.64mm_HandSolder
Connections:
- net GNDREF: now also C2.2, C3.2, BT1.2 (-), J1.2 (Pin_2), J2.2 (Pin_2), U1.1 (GND)
- net at C1.1, L1.2: now also J2.1 (Pin_1); no longer C3.1
- net at Q1.1 (D): now also J1.1 (Pin_1)
- net Signal: now reaches Q1.2 (G)
- net Signal: now also U1.3 (Q)
- net at C2.1: now also U1.5 (CV)
- net at R1.2: now also D2.2 (A), RV1.1, RV1.2
- net at R1.1: now also BT1.1 (+), U1.4 (R), U1.8 (VCC)
- new net: C3.1, D3.1 (K), RV1.3, U1.2 (TR), U1.6 (THR)
- new net: D2.1 (K), D3.2 (A), U1.7 (DIS)

Commit message: yol kalınlığı
projelerde pcb yol kalınlıkları akım kapasitelerine göre yeniden düzenlendi
Connections:
- net VCC: now reaches J1.1 (Pin_1), Q1.1 (D)
- net +5V: now reaches BT1.1 (+), R1.1, U1.4 (R), U1.8 (VCC)
Changed lines of the file:
@@
 	4300 4350 4300 3900
 Wire Wire Line
-	4300 3900 2650 3900
+	4300 3900 2850 3900
 Wire Wire Line
 	2650 3900 2650 4350
@@
 Connection ~ 8000 3050
 Wire Wire Line
-	5750 1950 5000 1950
+	5750 1950 5350 1950
 Wire Wire Line
 	5000 1950 5000 2100
@@
 Wire Wire Line
 	2650 5550 2650 5450
+$Comp
+L power:+5V #PWR0103
+U 1 1 6144746C
+P 2850 3800
+F 0 "#PWR0103" H 2850 3650 50  0001 C CNN
+F 1 "+5V" H 2865 3973 50  0000 C CNN
+F 2 "" H 2850 3800 50  0001 C CNN
+F 3 "" H 2850 3800 50  0001 C CNN
+	1    2850 3800
+	1    0    0    -1
+$EndComp
+Wire Wire Line
+	2850 3800 2850 3900
+Connection ~ 2850 3900
+Wire Wire Line
+	2850 3900 2650 3900
+$Comp
+L power:VCC #PWR0104
+U 1 1 61449E30
+P 5350 1850
+F 0 "#PWR0104" H 5350 1700 50  0001 C CNN
+F 1 "VCC" H 5365 2023 50  0000 C CNN
+F 2 "" H 5350 1850 50  0001 C CNN
+F 3 "" H 5350 1850 50  0001 C CNN
+	1    5350 1850
+	1    0    0    -1
+$EndComp
+Wire Wire Line
+	5350 1850 5350 1950
+Connection ~ 5350 1950
+Wire Wire Line
+	5350 1950 5000 1950
 $EndSCHEMATC
